File: Ashurs PCB/INTROmcu.kicad_sch (KiCad schematic)
At the start: 16 parts, among them U2 LMS8117AMP-3.3, U7 STM32G441KBT6

Commit message: post-david suggestions
u6 footprint, zener diode footprints, jumper footprints
Parts:
- D2, D5: footprint Diode_SMD:D_0201_0603Metric -> Diode_SMD:D_SOD-123F
- JP1, JP2: footprint Jumper:SolderJumper-2_P1.3mm_Bridged2Bar_Pad1.0x1.5mm -> Resistor_SMD:R_0201_0603Metric
Changed lines of the file:
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@@
 			)
 		)
-		(property "Footprint" "Diode_SMD:D_0201_0603Metric"
+		(property "Footprint" "Diode_SMD:D_SOD-123F"
 			(at 109.22 133.35 0)
 			(effects
@@
 			)
 		)
-		(property "Footprint" "Jumper:SolderJumper-2_P1.3mm_Bridged2Bar_Pad1.0x1.5mm"
+		(property "Footprint" "Resistor_SMD:R_0201_0603Metric"
 			(at 146.05 102.87 0)
 			(effects
@@
 			)
 		)
-		(property "Footprint" "Jumper:SolderJumper-2_P1.3mm_Bridged2Bar_Pad1.0x1.5mm"
+		(property "Footprint" "Resistor_SMD:R_0201_0603Metric"
 			(at 90.17 109.22 0)
 			(effects
@@
 			)
 		)
-		(property "Footprint" "Diode_SMD:D_0201_0603Metric"
+		(property "Footprint" "Diode_SMD:D_SOD-123F"
 			(at 109.22 128.27 0)
 			(effects

Commit message: footprint mistake
Parts:
- U2: footprint footprint:10LGA_2X2X0p75_BOS -> footprint:MP04A_TEX
Changed lines of the file:
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@@
 			)
 		)
-		(property "Footprint" "footprint:10LGA_2X2X0p75_BOS"
+		(property "Footprint" "footprint:MP04A_TEX"
 			(at 31.75 130.81 0)
 			(effects
